File: DesktopControl-HW/DesktopControl-HW.kicad_sch (KiCad schematic)
At the start: 8 parts

Commit message: Rework amplifier configuration, add amplifier for subwoofer and start check of codec
Parts:
- added C58, C59: 100n, symbol Device:C_Polarized
- added R16: 4k7, Resistor_SMD:R_0603_1608Metric_Pad0.98x0.95mm_HandSolder, symbol Device:R
- added R22, R23: 12k, Resistor_SMD:R_0603_1608Metric_Pad0.98x0.95mm_HandSolder, symbol Device:R
- added R24, R25: 47k, Resistor_SMD:R_0603_1608Metric_Pad0.98x0.95mm_HandSolder, symbol Device:R
Connections:
- net GND: now also C58.2, C59.2, R24.1, R25.1
- new net AMPLIFIER/SYNC: R16.2
- new net AMPLIFIER_SUB/AUDIO_L: C59.1, R22.2
- new net AMPLIFIER_SUB/AUDIO_R: C58.1, R23.2
- new net AMPLIFIER_SUB/SYNC: R16.1
- new net AUDIO_L: R22.1, R25.2
- new net AUDIO_R: R23.1, R24.2
Other:
- sheet AMPLIFIER_L renamed AMPLIFIER
- removed sheet AMPLIFIER_R
- removed sheet TRIANGLE_GEN
- added sheet AMPLIFIER_SUB (AMPLIFIER_SUB.kicad_sch)
- sheet AMPLIFIER ports: added AUDIO_L, AUDIO_R, MUTE, OUT_LN, OUT_LP, OUT_RN, OUT_RP, SYNC; removed AUDIO_IN, AUDIO_OUT, TRIANGLE
- note added: "AUDIO AMPLIFIERS"
- note added: "Fc = 132 Hz"
